File: simpleclock_v1.sch (EAGLE design)
At the start: 88 parts, among them IC1 TINY24/44/84-SSU

Commit message: wow, it's been that long since i committed?
Parts:
- added RDOWN, RUP: (no value), SparkFun:RESISTOR1206
Connections:
- net N$1 renamed PB2
- net N$2 renamed PA7
- net N$3 renamed PA6
- net N$4 renamed PA5
- net N$5 renamed PA4
- net N$6 renamed PA3
- net N$7 renamed PA2
- net N$8 renamed PA1
- net N$9 renamed PA0
- removed net N$10: IC1.(PCINT9/XTAL2)PB1
- removed net N$11: IC1.(PCINT8/XTAL1/CLKI)PB0
- removed net N$20: IC1.(PCINT11/RESET/DW)PB3, RESET.TP
- new net PB0: IC1.(PCINT8/XTAL1/CLKI)PB0, RUP.2
- new net PB1: IC1.(PCINT9/XTAL2)PB1, RDOWN.2
- new net PB3: IC1.(PCINT11/RESET/DW)PB3, RDOWN.1, RESET.TP, RUP.1
Changed lines of the file:
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@@
 <part name="GND" library="testpad" deviceset="PTR1" device="PAD1-13"/>
 <part name="SUPPLY3" library="supply2" deviceset="GND" device=""/>
+<part name="RUP" library="SparkFun" deviceset="RESISTOR" device="1206"/>
+<part name="RDOWN" library="SparkFun" deviceset="RESISTOR" device="1206"/>
 </parts>
 <sheets>
@@
 <instance part="GND" gate="G$1" x="302.26" y="68.58" rot="R90"/>
 <instance part="SUPPLY3" gate="GND" x="355.6" y="116.84"/>
+<instance part="RUP" gate="G$1" x="294.64" y="157.48"/>
+<instance part="RDOWN" gate="G$1" x="317.5" y="157.48"/>
 </instances>
 <busses>
@@
 </segment>
 </net>
-<net name="N$1" class="0">
+<net name="PB2" class="0">
 <segment>
 <pinref part="RN9" gate="G$1" pin="1"/>
@@
 </segment>
 </net>
-<net name="N$2" class="0">
+<net name="PA7" class="0">
 <segment>
 <pinref part="RN8" gate="G$1" pin="1"/>
@@
 </segment>
 </net>
-<net name="N$3" class="0">
+<net name="PA6" class="0">
 <segment>
 <pinref part="RN7" gate="G$1" pin="1"/>
@@
 </segment>
 </net>
-<net name="N$4" class="0">
+<net name="PA5" class="0">
 <segment>
 <pinref part="RN6" gate="G$1" pin="1"/>
@@
 </segment>
 </net>
-<net name="N$5" class="0">
+<net name="PA4" class="0">
 <segment>
 <pinref part="RN5" gate="G$1" pin="1"/>
@@
 </segment>
 </net>
-<net name="N$6" class="0">
+<net name="PA3" class="0">
 <segment>
 <pinref part="RN4" gate="G$1" pin="1"/>
@@
 </segment>
 </net>
-<net name="N$7" class="0">
+<net name="PA2" class="0">
 <segment>
 <pinref part="RN3" gate="G$1" pin="1"/>
@@
 </segment>
 </net>
-<net name="N$8" class="0">
+<net name="PA1" class="0">
 <segment>
 <pinref part="RN2" gate="G$1" pin="1"/>
@@
 </segment>
 </net>
-<net name="N$9" class="0">
+<net name="PA0" class="0">
 <segment>
 <pinref part="RN1" gate="G$1" pin="1"/>
@@
 </segment>
 </net>
-<net name="N$20" class="0">
+<net name="PB3" class="0">
 <segment>
 <pinref part="IC1" gate="1" pin="(PCINT11/RESET/DW)PB3"/>
@@
 <wire x1="340.36" y1="83.82" x2="340.36" y2="127" width="0.1524" layer="91"/>
 </segment>
-</net>
-<net name="N$10" class="0">
+<segment>
+<pinref part="RDOWN" gate="G$1" pin="1"/>
+<wire x1="312.42" y1="157.48" x2="312.42" y2="167.64" width="0.1524" layer="91"/>
+<pinref part="RUP" gate="G$1" pin="1"/>
+<wire x1="289.56" y1="157.48" x2="289.56" y2="167.64" width="0.1524" layer="91"/>
+<wire x1="312.42" y1="167.64" x2="289.56" y2="167.64" width="0.1524" layer="91"/>
+<wire x1="289.56" y1="167.64" x2="279.4" y2="167.64" width="0.1524" layer="91"/>
+<junction x="289.56" y="167.64"/>
+<label x="279.4" y="167.64" size="1.778" layer="95"/>
+</segment>
+</net>
+<net name="PB1" class="0">
 <segment>
 <pinref part="IC1" gate="1" pin="(PCINT9/XTAL2)PB1"/>
 <wire x1="330.2" y1="121.92" x2="342.9" y2="121.92" width="0.1524" layer="91"/>
 </segment>
-</net>
-<net name="N$11" class="0">
+<segment>
+<pinref part="RDOWN" gate="G$1" pin="2"/>
+<wire x1="322.58" y1="157.48" x2="322.58" y2="147.32" width="0.1524" layer="91"/>
+<label x="322.58" y="144.78" size="1.778" layer="95"/>
+</segment>
+</net>
+<net name="PB0" class="0">
 <segment>
 <pinref part="IC1" gate="1" pin="(PCINT8/XTAL1/CLKI)PB0"/>
 <wire x1="330.2" y1="119.38" x2="342.9" y2="119.38" width="0.1524" layer="91"/>
+</segment>
+<segment>
+<pinref part="RUP" gate="G$1" pin="2"/>
+<wire x1="299.72" y1="157.48" x2="299.72" y2="147.32" width="0.1524" layer="91"/>
+<label x="299.72" y="144.78" size="1.778" layer="95"/>
 </segment>
 </net>
@@
 </sheet>
 </sheets>
+<errors>
+</errors>
 </schematic>
 </drawing>

Commit message: new board outline
Parts:
- added IC2: MEGA48/88/168-AU, avr-7:MEGA48/88/168-AU
Changed lines of the file:
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@@
 <part name="RUP" library="SparkFun" deviceset="RESISTOR" device="1206"/>
 <part name="RDOWN" library="SparkFun" deviceset="RESISTOR" device="1206"/>
+<part name="IC2" library="avr-7" deviceset="MEGA48/88/168" device="-AU"/>
 </parts>
 <sheets>
@@
 <instance part="RUP" gate="G$1" x="294.64" y="157.48"/>
 <instance part="RDOWN" gate="G$1" x="317.5" y="157.48"/>
+<instance part="IC2" gate="1" x="358.14" y="187.96"/>
 </instances>
 <busses>
