File: radiata_v1.sch (EAGLE design)
At the start: 128 parts, among them IC2 MEGA48/88/168-AU, Q1 FA-20H

Commit message: final versions of board and schematic
Parts:
- added C3: (no value), rcl:C-USC0603
- PNP1, PNP2, PNP3, PNP4, PNP5, PNP6, PNP7, PNP8, PNP9: device transistor:MMBT540LT1-PNP-SOT23-BEC -> transistor:MMBT2907ALT1-PNP-SOT23-BEC
- renumbered SCL to SCK
Connections:
- net GND: now also C3.2
- net VCC: now also C3.1
Changed lines of the file:
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@@
 <part name="MISO" library="testpad" deviceset="PTR1" device="TP19R" value="PTR1TP19R"/>
 <part name="MOSI" library="testpad" deviceset="PTR1" device="TP19R" value="PTR1TP19R"/>
-<part name="SCL" library="testpad" deviceset="PTR1" device="TP19R" value="PTR1TP19R"/>
+<part name="SCK" library="testpad" deviceset="PTR1" device="TP19R" value="PTR1TP19R"/>
 <part name="RESET" library="testpad" deviceset="PTR1" device="TP19R" value="PTR1TP19R"/>
 <part name="VCC" library="testpad" deviceset="PTR1" device="TP19R" value="PTR1TP19R"/>
@@
 <part name="V+" library="testpad" deviceset="PTR1" device="TP20SQ"/>
 <part name="NPN1" library="transistor" deviceset="*-NPN-" device="SOT23-BEC" technology="MMBT2222ALT1"/>
-<part name="PNP1" library="transistor" deviceset="*-PNP-" device="SOT23-BEC" technology="MMBT540LT1"/>
+<part name="PNP1" library="transistor" deviceset="*-PNP-" device="SOT23-BEC" technology="MMBT2907ALT1"/>
 <part name="CN1" library="rcl" deviceset="R-US_" device="M0805"/>
 <part name="SUPPLY1" library="supply2" deviceset="GND" device=""/>
@@
 <part name="P+4" library="supply1" deviceset="VCC" device=""/>
 <part name="NPN2" library="transistor" deviceset="*-NPN-" device="SOT23-BEC" technology="MMBT2222ALT1"/>
-<part name="PNP2" library="transistor" deviceset="*-PNP-" device="SOT23-BEC" technology="MMBT540LT1"/>
+<part name="PNP2" library="transistor" deviceset="*-PNP-" device="SOT23-BEC" technology="MMBT2907ALT1"/>
 <part name="CN2" library="rcl" deviceset="R-US_" device="M0805"/>
 <part name="SUPPLY6" library="supply2" deviceset="GND" device=""/>
 <part name="P+5" library="supply1" deviceset="VCC" device=""/>
 <part name="NPN3" library="transistor" deviceset="*-NPN-" device="SOT23-BEC" technology="MMBT2222ALT1"/>
-<part name="PNP3" library="transistor" deviceset="*-PNP-" device="SOT23-BEC" technology="MMBT540LT1"/>
+<part name="PNP3" library="transistor" deviceset="*-PNP-" device="SOT23-BEC" technology="MMBT2907ALT1"/>
 <part name="SUPPLY7" library="supply2" deviceset="GND" device=""/>
 <part name="CN3" library="rcl" deviceset="R-US_" device="M0805"/>
 <part name="NPN4" library="transistor" deviceset="*-NPN-" device="SOT23-BEC" technology="MMBT2222ALT1"/>
-<part name="PNP4" library="transistor" deviceset="*-PNP-" device="SOT23-BEC" technology="MMBT540LT1"/>
+<part name="PNP4" library="transistor" deviceset="*-PNP-" device="SOT23-BEC" technology="MMBT2907ALT1"/>
 <part name="CN4" library="rcl" deviceset="R-US_" device="M0805"/>
 <part name="SUPPLY8" library="supply2" deviceset="GND" device=""/>
@@
 <part name="P+7" library="supply1" deviceset="VCC" device=""/>
 <part name="NPN5" library="transistor" deviceset="*-NPN-" device="SOT23-BEC" technology="MMBT2222ALT1"/>
-<part name="PNP5" library="transistor" deviceset="*-PNP-" device="SOT23-BEC" technology="MMBT540LT1"/>
+<part name="PNP5" library="transistor" deviceset="*-PNP-" device="SOT23-BEC" technology="MMBT2907ALT1"/>
 <part name="CN5" library="rcl" deviceset="R-US_" device="M0805"/>
 <part name="SUPPLY9" library="supply2" deviceset="GND" device=""/>
 <part name="P+8" library="supply1" deviceset="VCC" device=""/>
 <part name="NPN6" library="transistor" deviceset="*-NPN-" device="SOT23-BEC" technology="MMBT2222ALT1"/>
-<part name="PNP6" library="transistor" deviceset="*-PNP-" device="SOT23-BEC" technology="MMBT540LT1"/>
+<part name="PNP6" library="transistor" deviceset="*-PNP-" device="SOT23-BEC" technology="MMBT2907ALT1"/>
 <part name="SUPPLY10" library="supply2" deviceset="GND" device=""/>
 <part name="CN6" library="rcl" deviceset="R-US_" device="M0805"/>
 <part name="NPN7" library="transistor" deviceset="*-NPN-" device="SOT23-BEC" technology="MMBT2222ALT1"/>
-<part name="PNP7" library="transistor" deviceset="*-PNP-" device="SOT23-BEC" technology="MMBT540LT1"/>
+<part name="PNP7" library="transistor" deviceset="*-PNP-" device="SOT23-BEC" technology="MMBT2907ALT1"/>
 <part name="CN7" library="rcl" deviceset="R-US_" device="M0805"/>
 <part name="SUPPLY11" library="supply2" deviceset="GND" device=""/>
@@
 <part name="P+10" library="supply1" deviceset="VCC" device=""/>
 <part name="NPN8" library="transistor" deviceset="*-NPN-" device="SOT23-BEC" technology="MMBT2222ALT1"/>
-<part name="PNP8" library="transistor" deviceset="*-PNP-" device="SOT23-BEC" technology="MMBT540LT1"/>
+<part name="PNP8" library="transistor" deviceset="*-PNP-" device="SOT23-BEC" technology="MMBT2907ALT1"/>
 <part name="CN8" library="rcl" deviceset="R-US_" device="M0805"/>
 <part name="SUPPLY12" library="supply2" deviceset="GND" device=""/>
 <part name="P+11" library="supply1" deviceset="VCC" device=""/>
 <part name="NPN9" library="transistor" deviceset="*-NPN-" device="SOT23-BEC" technology="MMBT2222ALT1"/>
-<part name="PNP9" library="transistor" deviceset="*-PNP-" device="SOT23-BEC" technology="MMBT540LT1"/>
+<part name="PNP9" library="transistor" deviceset="*-PNP-" device="SOT23-BEC" technology="MMBT2907ALT1"/>
 <part name="SUPPLY13" library="supply2" deviceset="GND" device=""/>
 <part name="CN9" library="rcl" deviceset="R-US_" device="M0805"/>
+<part name="C3" library="rcl" deviceset="C-US" device="C0603"/>
 </parts>
 <sheets>
@@
 <instance part="MISO" gate="G$1" x="220.98" y="139.7"/>
 <instance part="MOSI" gate="G$1" x="226.06" y="142.24"/>
-<instance part="SCL" gate="G$1" x="215.9" y="137.16"/>
+<instance part="SCK" gate="G$1" x="215.9" y="137.16"/>
 <instance part="RESET" gate="G$1" x="144.78" y="198.12" rot="R270"/>
 <instance part="VCC" gate="G$1" x="101.6" y="195.58" rot="R90"/>
@@
 <instance part="SUPPLY13" gate="GND" x="254" y="48.26"/>
 <instance part="CN9" gate="G$1" x="243.84" y="60.96"/>
+<instance part="C3" gate="G$1" x="149.86" y="154.94"/>
 </instances>
 <busses>
@@
 <wire x1="152.4" y1="167.64" x2="149.86" y2="167.64" width="0.1524" layer="91"/>
 <junction x="149.86" y="167.64"/>
+<pinref part="C3" gate="G$1" pin="1"/>
+<wire x1="149.86" y1="162.56" x2="149.86" y2="157.48" width="0.1524" layer="91"/>
+<junction x="149.86" y="162.56"/>
 </segment>
 <segment>
@@
 <wire x1="152.4" y1="142.24" x2="149.86" y2="142.24" width="0.1524" layer="91"/>
 <junction x="149.86" y="142.24"/>
+<pinref part="C3" gate="G$1" pin="2"/>
+<wire x1="149.86" y1="149.86" x2="149.86" y2="147.32" width="0.1524" layer="91"/>
+<junction x="149.86" y="147.32"/>
 </segment>
 <segment>
@@
 <net name="N$6" class="0">
 <segment>
-<pinref part="SCL" gate="G$1" pin="TP"/>
+<pinref part="SCK" gate="G$1" pin="TP"/>
 <pinref part="IC2" gate="1" pin="PB5(SCK/PCINT5)"/>
 <wire x1="215.9" y1="139.7" x2="213.36" y2="139.7" width="0.1524" layer="91"/>
